File: PCB/Hackpad/Hackpad.kicad_pcb (KiCad board)
At the start: 2 copper layers, 60 x 64.5 mm, 7 parts, among them SW1 SW_Push, SW2 SW_Push, SW3 SW_Push, SW4 SW_Push, SW5 SW_Push, SW6 SW_Push, U1 MOUDLE-SEEEDUINO-XIAO

Commit message: Finished
Routing:
- net Net-(U1-PA4_A1_D1): track 0.00 -> 30.2 mm
Changed lines of the file:
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@@
 			(outputformat 1)
 			(mirror no)
-			(drillshape 1)
+			(drillshape 0)
 			(scaleselection 1)
-			(outputdirectory "")
+			(outputdirectory "C:/Projects/Hardware/Hackpad/Hackpad/PRODUCTION/gerber/")
 		)
 	)
@@
 	)
 	(segment
+		(start 144.5 78.673654)
+		(end 135.176346 69.35)
+		(width 0.2)
+		(layer "F.Cu")
+		(net "Net-(U1-PA4_A1_D1)")
+	)
+	(segment
+		(start 131.25 68.276346)
+		(end 131.25 60.503654)
+		(width 0.2)
+		(layer "F.Cu")
+		(net "Net-(U1-PA4_A1_D1)")
+	)
+	(segment
+		(start 132.323654 69.35)
+		(end 131.25 68.276346)
+		(width 0.2)
+		(layer "F.Cu")
+		(net "Net-(U1-PA4_A1_D1)")
+	)
+	(segment
+		(start 144.5 79)
+		(end 144.5 78.673654)
+		(width 0.2)
+		(layer "F.Cu")
+		(net "Net-(U1-PA4_A1_D1)")
+	)
+	(segment
+		(start 133.713654 58.04)
+		(end 134.75 58.04)
+		(width 0.2)
+		(layer "F.Cu")
+		(net "Net-(U1-PA4_A1_D1)")
+	)
+	(segment
+		(start 131.25 60.503654)
+		(end 133.713654 58.04)
+		(width 0.2)
+		(layer "F.Cu")
+		(net "Net-(U1-PA4_A1_D1)")
+	)
+	(segment
+		(start 135.176346 69.35)
+		(end 132.323654 69.35)
+		(width 0.2)
+		(layer "F.Cu")
+		(net "Net-(U1-PA4_A1_D1)")
+	)
+	(segment
